Commit message: IMU Sensor Fusion

File: src/my_robot_model/urdf/my_robo_simulation_imu.urdf (robot description, URDF)
Before this commit: robot robot, 8 links, 7 joints
Links:
- added link imu_link, mass 0.0093378; collision box size=0.05 0.01 0.02; visual box size=0.05 0.01 0.02
Joints:
- added joint imu_joint: type fixed, parent base_link, child imu_link, origin xyz=0.0075 0.0 0.25 rpy=0 0 3.14, axis 0 0 0
